File: Z80Breakout/kicad/Z80Breakout.kicad_sch (KiCad schematic)
At the start: 4 parts, among them J1 Pin1:20, J2 Pin21:40, J3 Host Z80, U1 Z80CPU

Commit message: Z80 Breakout
Parts:
- added TP1: GND, TestPoint:TestPoint_THTPad_D2.0mm_Drill1.0mm, symbol Connector:TestPoint
- added TP2: +5V, TestPoint:TestPoint_THTPad_D2.0mm_Drill1.0mm, symbol Connector:TestPoint
Connections:
- net GND: now also TP1.1
- net VCC: now also TP2.1
Changed lines of the file:
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@@
   (title_block
     (title "Z80 Breakout Board")
-    (date "2024-03-31")
-    (rev "1.0")
+    (date "2024-04-13")
+    (rev "1.3")
   )
   (junction (at 185.42 71.12) (diameter 0) (color 0 0 0 0)
@@
   (junction (at 185.42 81.28) (diameter 0) (color 0 0 0 0)
   )
+  (junction (at 115.57 46.99) (diameter 0) (color 0 0 0 0)
+  )
   (junction (at 204.47 81.28) (diameter 0) (color 0 0 0 0)
   )
@@
   (junction (at 185.42 78.74) (diameter 0) (color 0 0 0 0)
   )
+  (junction (at 115.57 123.19) (diameter 0) (color 0 0 0 0)
+  )
   (junction (at 185.42 83.82) (diameter 0) (color 0 0 0 0)
   )
@@
     (stroke (width 0) (type default))
   )
+  (wire (pts (xy 115.57 46.99) (xy 127 46.99))
+    (stroke (width 0) (type default))
+  )
   (wire (pts (xy 185.42 82.55) (xy 185.42 83.82))
     (stroke (width 0) (type default))
@@
     (stroke (width 0) (type default))
   )
+  (wire (pts (xy 127 46.99) (xy 127 41.91))
+    (stroke (width 0) (type default))
+  )
   (wire (pts (xy 204.47 95.25) (xy 204.47 96.52))
     (stroke (width 0) (type default))
@@
     (stroke (width 0) (type default))
   )
+  (wire (pts (xy 101.6 123.19) (xy 101.6 127))
+    (stroke (width 0) (type default))
+  )
   (wire (pts (xy 185.42 83.82) (xy 190.5 83.82))
     (stroke (width 0) (type default))
@@
     (stroke (width 0) (type default))
   )
+  (wire (pts (xy 115.57 123.19) (xy 101.6 123.19))
+    (stroke (width 0) (type default))
+  )
   (wire (pts (xy 209.55 85.09) (xy 204.47 85.09))
     (stroke (width 0) (type default))
@@
     (property "Intersheetrefs" "${INTERSHEET_REFS}" (at 139.1886 80.01 0)
       (effects (font (size 1.27 1.27)) (justify left) hide)
+    )
+  )
+  (symbol (lib_id "Connector:TestPoint") (at 127 41.91 0) (unit 1)
+    (in_bom yes) (on_board yes) (dnp no) (fields_autoplaced)
+    (property "Reference" "TP2" (at 129.54 37.338 0)
+      (effects (font (size 1.27 1.27)) (justify left))
+    )
+    (property "Value" "+5V" (at 129.54 39.878 0)
+      (effects (font (size 1.27 1.27)) (justify left))
+    )
+    (property "Footprint" "TestPoint:TestPoint_THTPad_D2.0mm_Drill1.0mm" (at 132.08 41.91 0)
+      (effects (font (size 1.27 1.27)) hide)
+    )
+    (property "Datasheet" "~" (at 132.08 41.91 0)
+      (effects (font (size 1.27 1.27)) hide)
+    )
+    (pin "1")
+    (instances
+      (project "Z80Breakout"
+        (path "/717456a7-4132-4c36-bdf5-84a16b65bf79"
+          (reference "TP2") (unit 1)
+        )
+      )
     )
   )
@@
     )
   )
+  (symbol (lib_id "Connector:TestPoint") (at 101.6 127 180) (unit 1)
+    (in_bom yes) (on_board yes) (dnp no) (fields_autoplaced)
+    (property "Reference" "TP1" (at 104.14 129.032 0)
+      (effects (font (size 1.27 1.27)) (justify right))
+    )
+    (property "Value" "GND" (at 104.14 131.572 0)
+      (effects (font (size 1.27 1.27)) (justify right))
+    )
+    (property "Footprint" "TestPoint:TestPoint_THTPad_D2.0mm_Drill1.0mm" (at 96.52 127 0)
+      (effects (font (size 1.27 1.27)) hide)
+    )
+    (property "Datasheet" "~" (at 96.52 127 0)
+      (effects (font (size 1.27 1.27)) hide)
+    )
+    (pin "1")
+    (instances
+      (project "Z80Breakout"
+        (path "/717456a7-4132-4c36-bdf5-84a16b65bf79"
+          (reference "TP1") (unit 1)
+        )
+      )
+    )
+  )
   (symbol (lib_id "CPU:Z80CPU") (at 115.57 85.09 0) (unit 1)
-    (in_bom yes) (on_board yes) (dnp no) (fields_autoplaced)
-    (property "Reference" "U1" (at 117.7641 45.72 0)
+    (in_bom yes) (on_board yes) (dnp no)
+    (property "Reference" "U1" (at 102.87 49.53 0)
       (effects (font (size 1.27 1.27)) (justify left))
     )
