File: Z80Breakout/kicad/Z80Breakout.kicad_sch (KiCad schematic)
At the start: 6 parts, among them J1 Pin1:20, J2 Pin21:40, J3 Host Z80, U1 Z80CPU

Commit message: Kicad 9 updates
Parts:
- U1: footprint Package_DIP:DIP-40_W15.24mm -> 80bus:DIP-40_W15.24mm_ZIF
Other:
- title: Z80 Breakout Board -> Z80 Breakout Board - Kicad 9
Changed lines of the file:
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@@
 (kicad_sch
-	(version 20231120)
+	(version 20250114)
 	(generator "eeschema")
-	(generator_version "8.0")
+	(generator_version "9.0")
 	(paper "A4")
 	(title_block
-		(title "Z80 Breakout Board")
-		(date "2024-04-13")
-		(rev "1.3")
+		(title "Z80 Breakout Board - Kicad 9")
+		(date "2025-04-26")
+		(rev "1.5")
 	)
 	(junction
@@
 			)
 		)
-		(property "Description" ""
+		(property "Description" "test point"
 			(at 127 41.91 0)
 			(effects
@@
 			)
 		)
-		(property "Description" ""
+		(property "Description" "Special symbol for telling ERC where power comes from"
 			(at 120.65 123.19 0)
 			(effects
@@
 			)
 		)
-		(property "Description" ""
+		(property "Description" "Special symbol for telling ERC where power comes from"
 			(at 110.49 46.99 0)
 			(effects
@@
 			)
 		)
-		(property "Description" ""
+		(property "Description" "Generic connector, single row, 01x20, script generated"
 			(at 171.45 86.36 0)
 			(effects
@@
 			)
 		)
-		(property "Description" ""
+		(property "Description" "Generic connector, single row, 01x20, script generated"
 			(at 220.98 86.36 0)
 			(effects
@@
 			)
 		)
-		(property "Description" ""
+		(property "Description" "test point"
 			(at 101.6 127 0)
 			(effects
@@
 			)
 		)
-		(property "Footprint" "Package_DIP:DIP-40_W15.24mm"
+		(property "Footprint" "80bus:DIP-40_W15.24mm_ZIF"
 			(at 115.57 74.93 0)
 			(effects
@@
 			)
 		)
-		(property "Description" ""
+		(property "Description" "8-bit General Purpose Microprocessor, DIP-40"
 			(at 115.57 85.09 0)
 			(effects
@@
 			)
 		)
-		(property "Description" ""
+		(property "Description" "Generic connector, double row, 02x20, counter clockwise pin numbering scheme (similar to DIP package numbering), script generated (kicad-library-utils/schlib/autogen/connector/)"
 			(at 195.58 86.36 0)
 			(effects
@@
 		)
 	)
+	(embedded_fonts no)
 )
