File: Z80Breakout/kicad/Z80Breakout.kicad_pcb (KiCad board)
At the start: 2 copper layers, 58 x 60 mm, 9 parts, among them J1 Pin1:20, J2 Pin21:40, J3 Host Z80, U1 Z80CPU

Commit message: Kicad 9 updates
Parts:
- U1: footprint Package_DIP:DIP-40_W15.24mm -> 80bus:DIP-40_W15.24mm_ZIF
Other:
- board text added: "Ver 1.5"
- board text added: "fb1bdc30-9a17-4464-a638-e00785921f6e"
- board text removed: "34978414-f51e-4b87-8ded-4959e16cafcc"
- board text removed: "Ver 1.4"

Commit message: Minor changes
Other:
- board text added: "CS-007"
- board text removed: "CS-002"
Changed lines of the file:
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@@
 		)
 	)
-	(gr_text "CS-002"
+	(gr_text "CS-007"
 		(at 115.65216 108.286691 0)
 		(layer "F.SilkS")
