File: N1Clock/kicad/N1Clock.kicad_pcb (KiCad board)
At the start: 2 copper layers, 40 x 26 mm, 4 parts, among them X1 AEL1200CS

Commit message: Kicad 9 updates
Other:
- board text added: "Version 1.1"
- board text removed: "Version 1.0.0"
