File: N1Clock/kicad/N1Clock.kicad_sch (KiCad schematic)
At the start: 4 parts, among them X1 AEL1200CS

Commit message: Kicad 9 updates
Other:
- title: Nascom 1 Replacement Clock -> Nascom 1 Replacement Clock - Kicad 9
