File: N1Graphics/kicad/N1Graphics.kicad_pcb (KiCad board)
At the start: 2 copper layers, 29 x 38.2 mm, 4 parts, among them J1 D7 Output, U1 Character_ROM, U2 27C32

Commit message: Kicad 9 updates
Parts:
- removed G***: LOGO, LOGO
- added G001: LOGO, 80bus:sleepymouse_tiny, F.Cu at (120.9, 71.7)
- added G002: LOGO, 80bus:sleepymouse_tiny, F.Cu at (121.1, 56.1)
- J1: value D7 Output -> Conn_01x01_Pin
Connections:
- U1 pad 1: (no net) -> unconnected-(U1-Vbb-Pad1)
- U1 pad 10: (no net) -> unconnected-(U1-NC-Pad10)
- U1 pad 22: Net-(U1-Pad22) -> Net-(U1-RS1)
- U1 pad 24: Net-(U1-Pad24) -> Net-(U1-RS1)
- U1 pad 3: (no net) -> unconnected-(U1-Vdd-Pad3)
- U2 pad 5: Net-(U1-Pad24) -> Net-(U1-RS1)
- U2 pad 7: Net-(U1-Pad22) -> Net-(U1-RS1)
Routing:
- net Net-(U1-RS1): track 0.00 -> 30.9 mm
- net Net-(U1-Pad24): track 15.4 -> 0.00 mm
- net Net-(U1-Pad22): track 15.4 -> 0.00 mm
Other:
- board text added: "Graphics ROM data held in a 2732 Original data -> 0x0000 to 0x07FF Graphics Data -> 0x0800 to 0x0FFF"
- board text added: "Nascom 1 Add on Graphics"
- board text added: "Nascom 1 Graphics Extension Ver 2.2"
- board text added: "b462e7a9-32d1-430a-a488-a22e83f8ba13"
- board text removed: "0fedd434-39fa-4f8e-88e7-81edb081c40a"
- board text removed: "Nascom 1 Add on Graphics Graphics ROM data held in a 2732 Original data -> 0x0000 to 0x07FF Graphics Data -> 0x0800 to 0x0FFF"
- board text removed: "Nascom 1 Graphics Extension Ver 2.1"

Commit message: Minor changes
Other:
- board text added: "CS-009"
Changed lines of the file:
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@@
+		)
+	)
+	(gr_text "CS-009"
+		(at 122.95547 46.08575 0)
+		(layer "B.SilkS")
+		(effects
+			(font
+				(size 1 1)
+				(thickness 0.25)
+			)
+			(justify mirror)
 		)
 	)
