File: N1KeyAdaptor/kicad/N1KeyAdaptor.kicad_pcb (KiCad board)
At the start: 2 copper layers, 14.6 x 25.4 mm, 3 parts, among them J1 Nas 1 KBD, J2 NAS 2 KBD

Commit message: Kicad 9 updates
Parts:
- renumbered G*** to G001
Connections:
- J1 pad 15: (no net) -> unconnected-(J1-Pin_15-Pad15)
- J2 pad 4: (no net) -> unconnected-(J2-Pin_4-Pad4)
Other:
- board text added: "V2.2"
- board text removed: "V2.1.0"
