File: N1KeyAdaptor/kicad/N1KeyAdaptor.kicad_sch (KiCad schematic)
At the start: 2 parts, among them J1 Nas 1 KBD, J2 NAS 2 KBD

Commit message: Kicad 9 updates
Other:
- title: N1 Keyboard Adaptor -> N1 Keyboard Adaptor - Kicad 9
