File: N2ScreenFlashEliminator/kicad/N2Graphics.kicad_sch (KiCad schematic)
At the start: 13 parts, among them J1 Header, Q1 BC557, SW1 Cap Enable, SW2 Unit Enable, U1 74LS00, U2 74LS74, U3 74LS32

Commit message: Docs
Other:
- note added: "Connections Unit replaces IC69 (74LS32) TP1 - IC1/24 (Useable TPH near IC7) TP2 - IC67/11 (Usable TPH near IC67) Remove IC58 (Snowplough) (74LS123)"
- note removed: "Connections Unit replaces IC69 (74LS32) TP1 - IC1/24 (Useable TPH near ear IC7) TP2 - IC67/11 (Usable TPH near IC67) Remove IC58 (Snowplough) (74LS123)"
Changed lines of the file:
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@@
     (stroke (width 0) (type default))
   )
-  (text "Connections\n\nUnit replaces IC69 (74LS32)\n\nTP1 - IC1/24 (Useable TPH near ear IC7)\n\nTP2 - IC67/11 (Usable TPH near IC67)\n\nRemove IC58 (Snowplough) (74LS123)\n\n\n\n\n\n"
+  (text "Connections\n\nUnit replaces IC69 (74LS32)\n\nTP1 - IC1/24 (Useable TPH near IC7)\n\nTP2 - IC67/11 (Usable TPH near IC67)\n\nRemove IC58 (Snowplough) (74LS123)\n\n\n\n\n\n"
     (at 27.94 158.75 0)
     (effects (font (size 1.27 1.27)) (justify left bottom))

Commit message: Kicad 9 updates
Other:
- title: N2 Screen Flash Eliminator -> N2 Screen Flash Eliminator - Kicad 9
