File: lipoGardenLightCompact/kicad/lipoGardenLight.kicad_sch (KiCad schematic)
At the start: 14 parts, among them Q1 BC557, Q2 SS8050, Q3 SS8050

Commit message: Kicad 9 updates
Parts:
- Q1, Q2, Q3: footprint Package_TO_SOT_THT:TO-92_Wide -> Package_TO_SOT_THT:TO-92_Inline_Wide
Other:
- title: Lipo Solar Garden Light -> Lipo Solar Garden Light - Kicad 9
Changed lines of the file:
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@@
 (kicad_sch
-	(version 20231120)
+	(version 20250114)
 	(generator "eeschema")
-	(generator_version "8.0")
+	(generator_version "9.0")
 	(paper "A4")
 	(title_block
-		(title "Lipo Solar Garden Light")
-		(date "2021-12-26")
-		(rev "1.4")
+		(title "Lipo Solar Garden Light - Kicad 9")
+		(date "2025-04-26")
+		(rev "1.6")
 	)
 	(junction
@@
 			)
 		)
-		(property "Description" ""
+		(property "Description" "Single solar cell"
 			(at 241.3 97.79 0)
 			(effects
@@
 			)
 		)
-		(property "Description" ""
+		(property "Description" "Single-cell battery"
 			(at 190.5 97.79 0)
 			(effects
@@
 			)
 		)
-		(property "Description" ""
+		(property "Description" "Power symbol creates a global label with name \"GND\" , ground"
 			(at 135.89 88.9 0)
 			(effects
@@
 			)
 		)
-		(property "Description" ""
+		(property "Description" "40V 1A Schottky Barrier Rectifier Diode, DO-41"
 			(at 190.5 81.28 0)
 			(effects
@@
 			)
 		)
-		(property "Description" ""
+		(property "Description" "Resistor"
 			(at 101.6 72.39 0)
 			(effects
@@
 			)
 		)
-		(property "Description" ""
+		(property "Description" "Power symbol creates a global label with name \"GND\" , ground"
 			(at 128.27 46.99 0)
 			(effects
@@
 			)
 		)
-		(property "Description" ""
+		(property "Description" "Power symbol creates a global label with name \"GND\" , ground"
 			(at 153.67 46.99 0)
 			(effects
@@
 			)
 		)
-		(property "Description" ""
+		(property "Description" "Resistor"
 			(at 190.5 60.96 0)
 			(effects
@@
 			)
 		)
-		(property "Description" ""
+		(property "Description" "Power symbol creates a global label with name \"GND\" , ground"
 			(at 190.5 106.68 0)
 			(effects
@@
 			)
 		)
-		(property "Description" ""
+		(property "Description" "Power symbol creates a global label with name \"GND\" , ground"
 			(at 241.3 106.68 0)
 			(effects
@@
 			)
 		)
-		(property "Description" ""
+		(property "Description" "Power symbol creates a global label with name \"GND\" , ground"
 			(at 190.5 46.99 0)
 			(effects
@@
 			)
 		)
-		(property "Description" ""
+		(property "Description" "Resistor"
 			(at 173.99 59.69 0)
 			(effects
@@
 			)
 		)
-		(property "Description" ""
+		(property "Description" "Light emitting diode"
+			(at 132.08 83.82 0)
+			(effects
+				(font
+					(size 1.27 1.27)
+				)
+				(hide yes)
+			)
+		)
+		(property "Sim.Pins" "1=K 2=A"
 			(at 132.08 83.82 0)
 			(effects
@@
 			)
 		)
-		(property "Description" ""
+		(property "Description" "Resistor"
 			(at 146.05 76.2 0)
 			(effects
@@
 			)
 		)
-		(property "Description" ""
+		(property "Description" "Resistor"
 			(at 119.38 83.82 0)
 			(effects
@@
 			)
 		)
-		(property "Footprint" "Package_TO_SOT_THT:TO-92_Wide"
+		(property "Footprint" "Package_TO_SOT_THT:TO-92_Inline_Wide"
 			(at 125.73 59.055 0)
 			(effects
@@
 			)
 		)
-		(property "Footprint" "Package_TO_SOT_THT:TO-92_Wide"
+		(property "Footprint" "Package_TO_SOT_THT:TO-92_Inline_Wide"
 			(at 151.13 53.975 0)
 			(effects
@@
 			)
 		)
-		(property "Footprint" "Package_TO_SOT_THT:TO-92_Wide"
+		(property "Footprint" "Package_TO_SOT_THT:TO-92_Inline_Wide"
 			(at 111.76 97.155 0)
 			(effects
@@
 			)
 		)
-		(property "Datasheet" "http://www.fairchildsemi.com/ds/BC/BC557.pdf"
+		(property "Datasheet" "https://www.onsemi.com/pub/Collateral/BC556BTA-D.pdf"
 			(at 106.68 95.25 0)
 			(effects
@@
 			)
 		)
-		(property "Description" ""
+		(property "Description" "0.1A Ic, 45V Vce, PNP Small Signal Transistor, TO-92"
 			(at 106.68 95.25 0)
 			(effects
@@
 			)
 		)
-		(property "Description" ""
+		(property "Description" "Resistor"
 			(at 241.3 81.28 0)
 			(effects
@@
 			)
 		)
-		(property "Description" ""
+		(property "Description" "Power symbol creates a global label with name \"GND\" , ground"
 			(at 215.9 106.68 0)
 			(effects
@@
 			)
 		)
-		(property "Description" ""
+		(property "Description" "1300mW Silicon planar power Zener diodes, DO-41"
 			(at 215.9 81.28 0)
 			(effects
@@
 		)
 	)
+	(embedded_fonts no)
 )
